Commit message: commit sim

File: urdf/storm_robot.urdf.xacro (robot description, xacro)
@@ -1,5 +1,4 @@
 <?xml version="1.0"?>
 <robot name="storm_robot" xmlns:xacro="http://www.ros.org/wiki/xacro">
-  <xacro:include filename="$(find velodyne_description)/urdf/VLP-16.urdf.xacro"/>
   <!-- ===== Links ===== -->
   <link name="base_footprint"/>
@@ -69,12 +68,12 @@
     <axis xyz="0 1 0"/>
   </joint>
-  <!-- Caster (passive front wheel for stability) -->
+  <!-- Caster — fixed box instead of sphere to avoid DART physics assertion -->
   <link name="caster_link">
     <visual>
-      <geometry><sphere radius="0.05"/></geometry>
+      <geometry><box size="0.1 0.1 0.1"/></geometry>
       <material name="grey"/>
     </visual>
     <collision>
-      <geometry><sphere radius="0.05"/></geometry>
+      <geometry><box size="0.1 0.1 0.1"/></geometry>
     </collision>
     <inertial>
@@ -88,14 +87,48 @@
     <origin xyz="0.25 0 -0.1" rpy="0 0 0"/>
   </joint>
-  <!-- VLP-16: mounted 0.876m above base_link to match real hardware offset -->
-  <xacro:VLP-16 parent="base_link" name="velodyne" topic="/velodyne_points"
-                hz="10" samples="1800" gpu="true">
+  <!-- VLP-16: mounting plate -->
+  <link name="velodyne_base_link">
+    <visual>
+      <origin xyz="0 0 0" rpy="0 0 0"/>
+      <geometry><cylinder radius="0.0516" length="0.0717"/></geometry>
+      <material name="dark_grey"><color rgba="0.2 0.2 0.2 1"/></material>
+    </visual>
+    <collision>
+      <origin xyz="0 0 0" rpy="0 0 0"/>
+      <geometry><cylinder radius="0.0516" length="0.0717"/></geometry>
+    </collision>
+    <inertial>
+      <mass value="0.1"/>
+      <inertia ixx="0.0001" ixy="0" ixz="0" iyy="0.0001" iyz="0" izz="0.0001"/>
+    </inertial>
+  </link>
+  <joint name="velodyne_base_mount_joint" type="fixed">
+    <parent link="base_link"/>
+    <child link="velodyne_base_link"/>
+    <!-- 0.876m matches the real hardware offset used in master_launch.py -->
     <origin xyz="0 0 0.876" rpy="0 0 0"/>
-  </xacro:VLP-16>
-  <!-- ===== Gazebo plugins ===== -->
-  <!-- Differential drive: publishes odom and odom->base_link TF -->
+  </joint>
+  <!-- VLP-16: sensor frame (origin of published point cloud) -->
+  <link name="velodyne">
+    <visual>
+      <origin xyz="0 0 0" rpy="0 0 0"/>
+      <geometry><cylinder radius="0.0516" length="0.0717"/></geometry>
+      <material name="dark_grey"/>
+    </visual>
+    <inertial>
+      <mass value="0.83"/>
+      <inertia ixx="0.000827" ixy="0" ixz="0" iyy="0.000827" iyz="0" izz="0.000827"/>
+    </inertial>
+  </link>
+  <joint name="velodyne_base_scan_joint" type="fixed">
+    <parent link="velodyne_base_link"/>
+    <child link="velodyne"/>
+    <origin xyz="0 0 0.03585" rpy="0 0 0"/>
+  </joint>
+  <!-- ===== Gazebo plugins (Ignition Fortress / ign-gazebo6 naming) ===== -->
+  <!-- Differential drive: publishes /odom and odom->base_link TF -->
   <gazebo>
-    <plugin filename="gz-sim-diff-drive-system"
-            name="gz::sim::systems::DiffDrive">
+    <plugin filename="ignition-gazebo-diff-drive-system"
+            name="ignition::gazebo::systems::DiffDrive">
       <left_joint>wheel_left_joint</left_joint>
       <right_joint>wheel_right_joint</right_joint>
@@ -114,22 +147,21 @@
     </plugin>
   </gazebo>
-  <!-- Joint state publisher: needed by robot_state_publisher -->
+  <!-- Joint state publisher: feeds robot_state_publisher -->
   <gazebo>
-    <plugin filename="gz-sim-joint-state-publisher-system"
-            name="gz::sim::systems::JointStatePublisher">
+    <plugin filename="ignition-gazebo-joint-state-publisher-system"
+            name="ignition::gazebo::systems::JointStatePublisher">
       <topic>joint_states</topic>
     </plugin>
   </gazebo>
-  <!-- Caster friction set to near-zero so it doesn't resist turning -->
+  <!-- Low friction on caster so it doesn't resist turning -->
   <gazebo reference="caster_link">
     <mu1>0.0</mu1>
     <mu2>0.0</mu2>
   </gazebo>
-  <!-- VLP16 GPU LiDAR sensor override: 16-beam, ±15°, 0.3–25m, 10Hz -->
+  <!-- VLP16 GPU LiDAR sensor: 16-beam, ±15°, 0.3–25m, 10Hz -->
   <gazebo reference="velodyne">
     <sensor name="vlp16" type="gpu_lidar">
       <topic>/velodyne_points</topic>
       <update_rate>10</update_rate>
-      <gz_frame_id>velodyne</gz_frame_id>
       <lidar>
         <scan>

Commit message: commit sim

File: urdf/storm_robot.urdf.xacro (robot description, xacro)
@@ -4,23 +4,25 @@
   <link name="base_footprint"/>
   <link name="base_link">
-    <visual>
-      <origin xyz="0 0 0" rpy="0 0 0"/>
+    <!-- Chassis offset upward so bottom sits above wheel axle, only wheels touch ground -->
+    <visual>
+      <origin xyz="0 0 0.15" rpy="0 0 0"/>
       <geometry><box size="0.6 0.4 0.3"/></geometry>
       <material name="grey"><color rgba="0.5 0.5 0.5 1"/></material>
     </visual>
     <collision>
-      <origin xyz="0 0 0" rpy="0 0 0"/>
+      <origin xyz="0 0 0.15" rpy="0 0 0"/>
       <geometry><box size="0.6 0.4 0.3"/></geometry>
     </collision>
     <inertial>
       <mass value="20.0"/>
-      <origin xyz="0 0 0"/>
+      <origin xyz="0 0 0.15"/>
       <inertia ixx="0.5" ixy="0" ixz="0" iyy="0.5" iyz="0" izz="0.5"/>
     </inertial>
   </link>
+  <!-- base_link origin is at wheel axle height (0.1m above ground) -->
   <joint name="base_footprint_joint" type="fixed">
     <parent link="base_footprint"/>
     <child link="base_link"/>
-    <origin xyz="0 0 0.15" rpy="0 0 0"/>
+    <origin xyz="0 0 0.1" rpy="0 0 0"/>
   </joint>
   <!-- Left wheel -->
@@ -43,5 +45,5 @@
     <parent link="base_link"/>
     <child link="wheel_left_link"/>
-    <origin xyz="0 0.2 -0.05" rpy="0 0 0"/>
+    <origin xyz="0 0.2 0" rpy="0 0 0"/>
     <axis xyz="0 1 0"/>
   </joint>
@@ -65,5 +67,5 @@
     <parent link="base_link"/>
     <child link="wheel_right_link"/>
-    <origin xyz="0 -0.2 -0.05" rpy="0 0 0"/>
+    <origin xyz="0 -0.2 0" rpy="0 0 0"/>
     <axis xyz="0 1 0"/>
   </joint>
@@ -89,8 +91,15 @@
   <!-- VLP-16: mounting plate -->
   <link name="velodyne_base_link">
+    <!-- LiDAR head -->
     <visual>
       <origin xyz="0 0 0" rpy="0 0 0"/>
       <geometry><cylinder radius="0.0516" length="0.0717"/></geometry>
       <material name="dark_grey"><color rgba="0.2 0.2 0.2 1"/></material>
+    </visual>
+    <!-- Mounting pole: spans from chassis top (0.3m above base_link) up to this link (0.876m above base_link) -->
+    <visual>
+      <origin xyz="0 0 -0.288" rpy="0 0 0"/>
+      <geometry><cylinder radius="0.025" length="0.576"/></geometry>
+      <material name="dark_grey"/>
     </visual>
     <collision>

Commit message: commit sim

File: urdf/storm_robot.urdf.xacro (robot description, xacro)
@@ -87,5 +87,5 @@
     <parent link="base_link"/>
     <child link="caster_link"/>
-    <origin xyz="0.25 0 -0.1" rpy="0 0 0"/>
+    <origin xyz="0.25 0 -0.05" rpy="0 0 0"/>
   </joint>
   <!-- VLP-16: mounting plate -->

Commit message: commit sim

File: urdf/storm_robot.urdf.xacro (robot description, xacro)
@@ -70,6 +70,6 @@
     <axis xyz="0 1 0"/>
   </joint>
-  <!-- Caster — fixed box instead of sphere to avoid DART physics assertion -->
-  <link name="caster_link">
+  <!-- Front caster -->
+  <link name="caster_front_link">
     <visual>
       <geometry><box size="0.1 0.1 0.1"/></geometry>
@@ -84,8 +84,27 @@
     </inertial>
   </link>
-  <joint name="caster_joint" type="fixed">
-    <parent link="base_link"/>
-    <child link="caster_link"/>
+  <joint name="caster_front_joint" type="fixed">
+    <parent link="base_link"/>
+    <child link="caster_front_link"/>
     <origin xyz="0.25 0 -0.05" rpy="0 0 0"/>
+  </joint>
+  <!-- Rear caster -->
+  <link name="caster_rear_link">
+    <visual>
+      <geometry><box size="0.1 0.1 0.1"/></geometry>
+      <material name="grey"/>
+    </visual>
+    <collision>
+      <geometry><box size="0.1 0.1 0.1"/></geometry>
+    </collision>
+    <inertial>
+      <mass value="0.5"/>
+      <inertia ixx="0.001" ixy="0" ixz="0" iyy="0.001" iyz="0" izz="0.001"/>
+    </inertial>
+  </link>
+  <joint name="caster_rear_joint" type="fixed">
+    <parent link="base_link"/>
+    <child link="caster_rear_link"/>
+    <origin xyz="-0.25 0 -0.05" rpy="0 0 0"/>
   </joint>
   <!-- VLP-16: mounting plate -->
@@ -164,6 +183,10 @@
     </plugin>
   </gazebo>
-  <!-- Low friction on caster so it doesn't resist turning -->
-  <gazebo reference="caster_link">
+  <!-- Zero friction on casters so they don't resist turning -->
+  <gazebo reference="caster_front_link">
+    <mu1>0.0</mu1>
+    <mu2>0.0</mu2>
+  </gazebo>
+  <gazebo reference="caster_rear_link">
     <mu1>0.0</mu1>
     <mu2>0.0</mu2>
